Commit message: Added new simple body instancing on the basis of template rendering.

File: src/iai_bullet_sim/data/urdf/template_single_mesh.urdf (robot description, URDF)
Before this commit: robot {{object_name}}, 1 links, 0 joints
Links:
- link object: mass None -> {{mass}}; geometry collision mesh filename={{collision_path}} scale={{scale}} {{scale}} {{scale}}; visual mesh filename={{mesh_path}} scale={{scale}} {{scale}} {{scale}}
