Commit message: Overhaul, fixes, and AGENTS.md to enable them to use this lib

File: src/prime_bullet/urdf/scale.urdf (robot description, URDF)
Before this commit: robot scale, 2 links, 1 joints
Links:
- link base: mass None -> 80; geometry collision mesh filename=package://prime_bullet/meshes/scale_base.dae; visual mesh filename=package://prime_bullet/meshes/scale_base.dae
- link plate: mass None -> 20; geometry collision mesh filename=package://prime_bullet/meshes/scale_plate.dae; visual mesh filename=package://prime_bullet/meshes/scale_plate.dae

File: src/prime_bullet/urdf/windmill.urdf (robot description, URDF)
Before this commit: robot windmill, 3 links, 2 joints
Links:
- link base: mass None -> 80; geometry collision mesh filename=package://prime_bullet/meshes/windmill_base.dae; visual mesh filename=package://prime_bullet/meshes/windmill_base.dae
- link head: mass None -> 20; geometry collision mesh filename=package://prime_bullet/meshes/windmill_head.dae; visual mesh filename=package://prime_bullet/meshes/windmill_head.dae
- link wings: mass None -> 4; geometry collision mesh filename=package://prime_bullet/meshes/windmill_wings.dae; visual mesh filename=package://prime_bullet/meshes/windmill_wings.dae
